File: PCB/MainShield/LeCoolStick-v1_1.brd (EAGLE design)
At the start: 55.5 x 55.9 mm, 14 parts

Commit message: Le Cool Stick - PCB V1.1
Parts:
- removed BLUETOOTH: 4P-2.0, Seeed-OPL-Connector:HW4-2.0
- removed JP3, JP4: (no value), pinhead:1X04
- removed U$1: ARDUINOMICRO, adafruit:ARDUINOMICRO
- added +5V, GND: (no value), LaCoolCo_Library:1X04
- added BT: 4P-2.0, LaCoolCo_Library:4P-2.0
- added PCB1: SHIELD_MICRO, LaCoolCo_Library:SHIELD_MICRO
- DHT, LUM: device Seeed-OPL-Connector:HW4-2.0 -> LaCoolCo_Library:4P-2.0
- H1, H2, H3, H4: value MOUNT-HOLE2.8 -> MOUNT-HOLEHOLE-2.8; device holes:2,8 -> LaCoolCo_Library:HOLE-2,8
- JP1, JP2: device pinhead:1X17 -> LaCoolCo_Library:1X17
- MOIST: device Seeed-OPL-Connector:HW4-2.0-90D -> LaCoolCo_Library:4P-2.0-90D
- X1: device con-ptr500:AK500/2 -> LaCoolCo_Library:AK500/2
- moved DHT 22.9 mm to (44.5, 12.7)
Connections:
- removed net N$1: JP2.9, MOIST.4, U$1.P$26
- removed net N$10: JP1.7, U$1.P$11
- removed net N$11: JP1.8, U$1.P$10
- removed net N$12: JP1.9, U$1.P$9
- removed net N$13: JP1.10, U$1.P$8
- removed net N$14: JP1.11, U$1.P$7
- removed net N$15: JP1.12, U$1.P$6
- removed net N$16: JP1.14, U$1.P$4
- removed net N$17: JP1.15, U$1.P$3
- removed net N$18: JP1.16, U$1.P$2
- removed net N$19: JP1.17, U$1.P$1
- removed net N$2: JP2.10, LUM.4, U$1.P$27
- removed net N$20: JP2.1, U$1.P$18
- removed net N$21: JP2.2, U$1.P$19
- removed net N$22: JP2.5, U$1.P$13
- removed net N$24: JP2.7, U$1.P$24
- removed net N$25: JP2.8, U$1.P$25
- removed net N$26: JP2.11, U$1.P$28
- removed net N$27: JP2.12, U$1.P$29
- removed net N$28: JP2.13, U$1.P$30
- removed net N$29: JP2.14, U$1.P$31
- removed net N$3: DHT.4, JP1.13, U$1.P$5
- removed net N$30: JP2.15, U$1.P$32
- removed net N$31: JP2.16, U$1.P$33
- removed net N$32: JP2.17, U$1.P$34
- removed net N$4: BLUETOOTH.4, JP1.4, U$1.P$14
- removed net N$5: BLUETOOTH.3, JP1.3, U$1.P$15
- removed net N$6: JP1.1, U$1.P$17
- removed net N$7: JP1.2, U$1.P$16
- removed net N$8: JP1.5, U$1.P$22
- new net 3.3V: JP2.16, PCB1.3V3
- new net A0-FREE: JP2.14, PCB1.A0
- new net A1-FREE: JP2.13, PCB1.A1
- new net A2-FREE: JP2.12, PCB1.A2
- new net A3-FREE: JP2.11, PCB1.A3
- new net A4-LUM: JP2.10, LUM.4, PCB1.A4
- new net A5-MOIST: JP2.9, MOIST.4, PCB1.A5
- new net AREF: JP2.15, PCB1.REF
- new net D0-RX1: JP1.4, PCB1.RX1
- new net D0-TX1: JP1.3, PCB1.TX1
- new net D10-FREE: JP1.15, PCB1.D10
- new net D11-FREE: JP1.16, PCB1.D11
- new net D12-FREE: JP1.17, PCB1.D12
- new net D13-FREE: JP2.17, PCB1.D13
- new net D2-DHT: DHT.4, JP1.7, PCB1.D2
- new net D3-FREE: JP1.8, PCB1.D3
- new net D4-FREE: JP1.9, PCB1.D4
- new net D5-FREE: JP1.10, PCB1.D5
- new net D6-FREE: JP1.11, PCB1.D6
- new net D7-FREE: JP1.12, PCB1.D7
- new net D8-BT(TX): BT.4, JP1.13, PCB1.D8
- new net D9-BT(RX): BT.3, JP1.14, PCB1.D9
- new net MISO-FREE: JP2.2, PCB1.MISO]
- new net MOSI-FREE: JP1.1, PCB1.MOSI
- new net N/C: JP2.8, PCB1.NC
- new net N/C.: JP2.7, PCB1.NC.
- new net RST: JP1.5, PCB1.RST
- new net RST.: JP2.5, PCB1.RST.
- new net SCK-FREE: JP2.1, PCB1.SCK
- new net SS-FREE: JP1.2, PCB1.SS
- net +5V: now also +5V.1, +5V.2, +5V.3, +5V.4, BT.2, PCB1.+5V; no longer BLUETOOTH.2, JP4.1, JP4.2, JP4.3, JP4.4, U$1.P$23
- net GND: now also BT.1, GND.1, GND.2, GND.3, GND.4, PCB1.GND, PCB1.GND.; no longer BLUETOOTH.1, JP3.1, JP3.2, JP3.3, JP3.4, U$1.P$12, U$1.P$21
- net VCC: now also PCB1.VIN; no longer U$1.P$20
Routing:
- net A5-MOIST: track 0.00 -> 26.2 mm
- net N$1: track 26.2 -> 0.00 mm
- net +5V: track 113.7 -> 136.9 mm
- net D2-DHT: track 0.00 -> 16.1 mm
- net A4-LUM: track 0.00 -> 13.5 mm
- net N$2: track 13.5 -> 0.00 mm
- net N$5: track 13.0 -> 0.00 mm
- net D9-BT(RX): track 0.00 -> 13.0 mm
- net N$3: track 8.44 -> 0.00 mm
- net N$4: track 8.43 -> 0.00 mm
- net D8-BT(TX): track 0.00 -> 8.43 mm
- net SCK-FREE: track 0.00 -> 3.81 mm
- net RST.: track 0.00 -> 3.81 mm
- net N/C.: track 0.00 -> 3.81 mm
- net N/C: track 0.00 -> 3.81 mm
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